Commit message: Working MiR with RGB-D Base_Cam. Added the 2 xacro files and deleted the old camera-things.

File: mir_description/urdf/include/mir_200.gazebo.xacro (robot description, xacro)
@@ -55,26 +55,3 @@
     </gazebo>
   </xacro:macro>
-    <!-- camera -->
-    <gazebo reference="camera_link">
-      <sensor type="depth" name="camera">
-        <plugin name="kinect_camera_controller" filename="libgazebo_ros_openni_kinect.so">
-          <cameraName>camera</cameraName>
-          <alwaysOn>true</alwaysOn>
-          <updateRate>10</updateRate>
-          <imageTopicName>rgb/image_raw</imageTopicName>
-          <depthImageTopicName>depth/image_raw</depthImageTopicName>
-          <pointCloudTopicName>depth/points</pointCloudTopicName>
-          <cameraInfoTopicName>rgb/camera_info</cameraInfoTopicName>
-          <depthImageCameraInfoTopicName>depth/camera_info</depthImageCameraInfoTopicName>
-          <frameName>camera_link_optical</frameName>
-          <baseline>0.1</baseline>
-          <distortion_k1>0.0</distortion_k1>
-          <distortion_k2>0.0</distortion_k2>
-          <distortion_k3>0.0</distortion_k3>
-          <distortion_t1>0.0</distortion_t1>
-          <distortion_t2>0.0</distortion_t2>
-          <pointCloudCutoff>0.4</pointCloudCutoff>
-        </plugin>
-      </sensor>
-    </gazebo>
 </robot>

File: mir_description/urdf/include/mir_200_v1.urdf.xacro (robot description, xacro)
@@ -9,4 +9,5 @@
   <xacro:include filename="$(find mir_description)/urdf/include/mir_200.transmission.xacro" />
   <xacro:include filename="$(find mir_description)/urdf/include/sick_s300.urdf.xacro" />
+  <xacro:include filename="$(find mir_description)/urdf/include/_d435.urdf.xacro"/>
   <xacro:property name="deg_to_rad" value="0.017453293" />
   <xacro:property name="mir_200_base_mass" value="58.0" />
@@ -211,44 +212,9 @@
     <link name="${prefix}surface"/>
     <xacro:mir_200_wheel_transmissions prefix="${prefix}"/>
-    <!-- disabled, because it doesn't make a difference in Gazebo: -->
-    <!-- <xacro:set_all_wheel_frictions prefix="${prefix}"/> -->
     <p3d_base_controller prefix="${prefix}" />
     <!-- Camera -->
-    <link name="camera_link">
-      <collision>
-        <origin xyz="0 0 0" rpy="0 0 0"/>
-        <geometry>
-          <box size="0.1 0.1 0.1"/>
-        </geometry>
-      </collision>
-      <visual>
-        <origin xyz="0 0 0" rpy="0 0 0"/>
-        <geometry>
-          <mesh filename="package://mir_description/meshes/visual/realsense.dae" />
-        </geometry>
-      </visual>
-      <inertial>
-        <mass value="1e-5" />
-        <origin xyz="0 0 0" rpy="0 0 0"/>
-        <inertia ixx="1e-6" ixy="0" ixz="0" iyy="1e-6" iyz="0" izz="1e-6" />
-      </inertial>
-    </link>
-    <joint name="camera_joint" type="fixed">
-      <axis xyz="0 1 0" />
-      <origin xyz="0.42 0 0.27" rpy="0 0.2 0"/> <!--set the position of the realsense-->
-      <parent link="${prefix}base_link"/>
-      <child link="camera_link"/>
-    </joint>
-    <!-- generate an optical frame http://www.ros.org/reps/rep-0103.html#suffix-frames
-        so that ros and opencv can operate on the camera frame correctly -->
-    <joint name="camera_optical_joint" type="fixed">
-      <!-- these values have to be these values otherwise the gazebo camera image
-          won't be aligned properly with the frame it is supposedly originating from -->
-      <origin xyz="0 0 0" rpy="-1.5708 0 -1.5708"/>
-      <parent link="camera_link"/>
-      <child link="camera_link_optical"/>
-    </joint>
-    <link name="camera_link_optical">
-    </link>
+    <xacro:sensor_d435 name="camera_base" parent="${prefix}base_link">
+      <origin xyz="0.42 0 0.27" rpy="0 0.2 0"/>
+    </xacro:sensor_d435>
   </xacro:macro>
 </robot>

File: mir_description/urdf/mir.urdf.xacro (robot description, xacro)
@@ -10,8 +10,4 @@
   <xacro:mir_200 prefix=""/>
   <xacro:controller_plugin_gazebo robot_namespace=""/>
-  <!-- Intel RealSense D435 PlugIn -->
-  <!--xacro:include filename="$(find mir_description)/urdf/include/_d435.urdf.xacro">
-    <sensor_d435 parent="${prefix}camera_link_optical"></sensor_d435>
-  </xacro:include-->
   <!-- instead of the controller_plugin_gazebo, you can use the diffdrive controller like this:
     <xacro:diff_controller_plugin_gazebo prefix=""
