Commit message: Added second RGB-D-Camera "on top" of Mir.

File: mir_description/urdf/include/mir_200_v1.urdf.xacro (robot description, xacro)
@@ -217,4 +217,7 @@
       <origin xyz="0.42 0 0.27" rpy="0 0.2 0"/>
     </xacro:sensor_d435>
+    <xacro:sensor_d435 name="camera_arm" parent="${prefix}base_link">
+      <origin xyz="0 0 1.0" rpy="0 0.2 0"/>
+    </xacro:sensor_d435>
   </xacro:macro>
 </robot>

Commit message: Added Arm_Controller and Transmissions to the "Fake_Arm" resulting in one rotational Freedom of the camera_arm.

File: mir_description/urdf/include/mir_200_v1.urdf.xacro (robot description, xacro)
@@ -213,10 +213,77 @@
     <xacro:mir_200_wheel_transmissions prefix="${prefix}"/>
     <p3d_base_controller prefix="${prefix}" />
+    <!--Fake Arm (z 0.450477) -->
+    <joint name="${prefix}robot_to_arm_joint" type="fixed">
+      <parent link="${prefix}base_link"/>
+      <child link="${prefix}arm_base_link"/>
+      <origin xyz="0.244311 -0.140242 0.39" rpy="0 0 0"/>
+    </joint>
+    <link name="${prefix}arm_base_link">
+      <visual>
+        <geometry>
+          <cylinder length="0.05" radius="0.07"/>
+        </geometry>
+        <material name="white"/>
+      </visual>
+      <collision>
+        <geometry>
+          <cylinder length="0.05" radius="0.07"/>
+        </geometry>
+      </collision>
+      <inertial>
+        <mass value="5"/>
+        <inertia ixx="0.007" ixy="0.0" ixz="0.0" iyy="0.007" iyz="0.0" izz="0.013"/>
+      </inertial>
+    </link>
+    <gazebo reference="${prefix}arm_base_link">
+      <material>Gazebo/LightGrey</material>
+      <selfCollide>true</selfCollide>
+    </gazebo>
+    <joint name="${prefix}arm_1_base_joint" type="continuous">
+      <parent link="${prefix}arm_base_link"/>
+      <child link="${prefix}arm_1_link"/>
+      <axis xyz="0 0 1"/>
+      <origin xyz="0 0 0.15" rpy="0 0 0"/>
+      <limit effort="30" velocity="1.0"/>
+      <dynamics damping="0.0" friction="0.0"/>
+    </joint>
+    <link name="${prefix}arm_1_link">
+      <visual>
+        <geometry>
+          <cylinder length="0.3" radius="0.05"/>
+        </geometry>
+        <material name="white"/>
+      </visual>
+      <collision>
+         <geometry>
+           <cylinder length="0.3" radius="0.05"/>
+        </geometry>
+      </collision>
+      <inertial>
+         <mass value="10"/>
+         <inertia ixx="0.08" ixy="0.0" ixz="0.0" iyy="0.08" iyz="0.0" izz="0.013"/>
+      </inertial>
+    </link>
+    <gazebo reference="${prefix}arm_1_link">
+      <material>Gazebo/LightGrey</material>
+      <selfCollide>true</selfCollide>
+    </gazebo>
+    <!-- transmission -->
+    <transmission name="base_to_arm_trans">
+      <type>transmission_interface/SimpleTransmission</type>
+      <actuator name="motorArm">
+        <hardwareInterface>hardware_interface/EffortJointInterface</hardwareInterface>
+        <mechanicalReduction>1</mechanicalReduction>
+      </actuator>
+      <joint name="${prefix}arm_1_base_joint">
+        <hardwareInterface>hardware_interface/EffortJointInterface</hardwareInterface>
+      </joint>
+    </transmission>
     <!-- Camera -->
     <xacro:sensor_d435 name="camera_base" parent="${prefix}base_link">
       <origin xyz="0.42 0 0.27" rpy="0 0.2 0"/>
     </xacro:sensor_d435>
-    <xacro:sensor_d435 name="camera_arm" parent="${prefix}base_link">
-      <origin xyz="0 0 1.0" rpy="0 0.2 0"/>
+    <xacro:sensor_d435 name="camera_arm" parent="${prefix}arm_1_link">
+      <origin xyz="0.025 0 0.16" rpy="0 0.2 0"/>
     </xacro:sensor_d435>
   </xacro:macro>

Commit message: Resized the Fake_Arm

File: mir_description/urdf/include/mir_200_v1.urdf.xacro (robot description, xacro)
@@ -251,5 +251,5 @@
       <visual>
         <geometry>
-          <cylinder length="0.3" radius="0.05"/>
+          <cylinder length="0.5" radius="0.05"/>
         </geometry>
         <material name="white"/>
@@ -257,5 +257,5 @@
       <collision>
          <geometry>
-           <cylinder length="0.3" radius="0.05"/>
+           <cylinder length="0.5" radius="0.05"/>
         </geometry>
       </collision>
@@ -285,5 +285,5 @@
     </xacro:sensor_d435>
     <xacro:sensor_d435 name="camera_arm" parent="${prefix}arm_1_link">
-      <origin xyz="0.025 0 0.16" rpy="0 0.2 0"/>
+      <origin xyz="0.025 0 0.26" rpy="0 0.2 0"/>
     </xacro:sensor_d435>
   </xacro:macro>

Commit message: Corrected Color Gazebo/LightGrey to White

File: mir_description/urdf/include/mir_200_v1.urdf.xacro (robot description, xacro)
@@ -152,5 +152,5 @@
     </link>
     <gazebo reference="${prefix}base_link">
-      <material>Gazebo/LightGrey</material>
+      <material>Gazebo/White</material>
     </gazebo>
     <!-- IMU -->
@@ -237,5 +237,5 @@
     </link>
     <gazebo reference="${prefix}arm_base_link">
-      <material>Gazebo/LightGrey</material>
+      <material>Gazebo/White</material>
       <selfCollide>true</selfCollide>
     </gazebo>
@@ -266,5 +266,5 @@
     </link>
     <gazebo reference="${prefix}arm_1_link">
-      <material>Gazebo/LightGrey</material>
+      <material>Gazebo/White</material>
       <selfCollide>true</selfCollide>
     </gazebo>
